File: Projecte_Seients.kicad_sch (KiCad schematic)
At the start: 43 parts, among them J1 Screw_Terminal_01x02, J2 Screw_Terminal_01x02, J3 Screw_Terminal_01x02, J4 Conn_01x05, J5 Conn_01x02, J6 Conn_01x03, J7 Conn_01x02, J8 Conn_01x05, J9 Conn_01x09, SW1 SW_Push, U1 LM1117DT-ADJ, U2 MCP2551-I-SN, U3 LM393, U4 PIC18F258, U5 24LC512, U6 DRV8871DDA, U7 DRV8871DDA, U8 DRV8871DDA, Y1 Crystal

Commit message: Add files via upload
Parts:
- removed U1: LM1117DT-ADJ, Mis_huellas:HuellaDis, symbol Regulator_Linear:LM1117DT-ADJ
- removed U4: PIC18F258, Package_SO:SOIC-28W_7.5x17.9mm_P1.27mm, symbol MCU_Microchip_PIC18:PIC18F2550-ISO
- removed U6, U7, U8: DRV8871DDA, Package_SO:Texas_HTSOP-8-1EP_3.9x4.9mm_P1.27mm_EP2.95x4.9mm_Mask2.4x3.1mm_ThermalVias, symbol Driver_Motor:DRV8871DDA
- added C10, C12: 100n, Capacitor_SMD:C_0805_2012Metric, symbol Device:C
- added C11, C13: 47n, Capacitor_SMD:C_0805_2012Metric, symbol Device:C
- added C14: 33n, Capacitor_SMD:C_0805_2012Metric, symbol Device:C
- added D10, D11, D5, D6, D7, D8: 1N5819, Diode_THT:D_DO-41_SOD81_P10.16mm_Horizontal, symbol Diode:1N5819
- added D9: D_TVS, Diode_THT:D_DO-41_SOD81_P7.62mm_Horizontal, symbol Device:D_TVS
- added J10, J13: Conn_01x03, symbol Connector_Generic:Conn_01x03
- added J11, J12: Conn_01x02, Connector_PinHeader_2.54mm:PinHeader_1x02_P2.54mm_Vertical, symbol Connector_Generic:Conn_01x02
- added J14: Screw_Terminal_01x02, symbol Connector:Screw_Terminal_01x02
- added K1: Relay_SPDT, symbol Relay:Relay_SPDT
- added Q1: DTC144E, symbol Transistor_BJT:DTC144E
- added R10, R11, R12, R15: 10k, Resistor_SMD:R_0805_2012Metric, symbol Device:R
- added R13, R14, R16, R17: 10k, Resistor_SMD:R_1206_3216Metric, symbol Device:R
- added R18: 1k, Resistor_SMD:R_0805_2012Metric, symbol Device:R
- added R19: 9k, Resistor_SMD:R_0805_2012Metric, symbol Device:R
- added R9: 0, Resistor_SMD:R_0805_2012Metric, symbol Device:R
- added SW2, SW3, SW4: SW_Push, symbol Switch:SW_Push
- added U10: PIC18F4580-IP, Package_DIP:DIP-40_W15.24mm, symbol MCU_Microchip_PIC18:PIC18F4580-IP
- added unit 2 of U3
- added U6, U9: L293D, Package_DIP:DIP-16_W7.62mm, symbol Driver_Motor:L293D
- added U7: LD1086V-DG, Package_TO_SOT_THT:TO-220-3_Vertical, symbol Regulator_Linear:LD1086V-DG
- added U8: LM393, symbol Comparator:LM393
- R5: value 1k -> 10k
Connections:
- net +5V: now also C9.2, R8.1, C12.2, J10.3 (Pin_3), J13.3 (Pin_3), R13.1, R16.1, U10.11 (VDD), U10.32 (VDD), U6.16 (VCC1), U7.2 (OUT), U8.8 (V+), U9.16 (VCC1); no longer C9.1
- net CANL: no longer C6.2, R1.2
- net GND: now also C9.1, C10.1, C12.1, C13.1, J10.1 (Pin_1), J11.1 (Pin_1), J12.1 (Pin_1), J13.1 (Pin_1), Q1.2 (E), R10.2, R11.2, R12.2, R14.2, R17.2, R18.2, R9.1, SW2.1, SW3.1, SW4.1, U10.12 (VSS), U10.31 (VSS), U6.12 (GND), U6.13 (GND), U6.4 (GND), U6.5 (GND), U8.4 (V-), U9.12 (GND), U9.13 (GND), U9.4 (GND), U9.5 (GND); no longer C9.2
- net PGC: now also U10.40 (RB7/KBI3/PGD)
- net PGD: now also U10.39 (RB6/KBI2/PGC)
- net PROG_MCLR: now also J6.1 (Pin_1); no longer J6.3 (Pin_3)
- net PWM: now also U10.18 (SCL/SCK/RC3), U6.1 (EN1,2), U9.1 (EN1,2), U9.9 (EN3,4)
- net RX: now also U10.26 (DT/RX/RC7)
- net RXCAN: now also U10.36 (RB3/CANRX)
- net SCL: now also U10.23 (SDA/SDI/RC4)
- net SDA: now also U5.5 (SDA), U10.24 (SDO/RC5)
- net TX: now also U10.25 (CK/TX/RC6)
- net TXCAN: now also U10.35 (RB2/INT2/CANTX)
- net VBAT: now also C11.2, C14.2, D10.1 (K), D5.1 (K), D7.1 (K), K1.11, K1.A1, U6.8 (VCC2), U9.8 (VCC2)
- net XTAL1: now also U10.14 (OSC2/CLKO/RA6)
- net XTAL2: now also U10.13 (OSC1/CLKI/RA7)
- net at J6.2 (Pin_2): now also U10.1 (~{MCLR}/VPP/RE3)
- net at C1.1, C2.1, D1.1 (K)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: now also U7.3 (IN)
- net at Cadj1.1, Radj1.2, Radj2.1: now also U7.1 (ADJ/GND)
- net M3_OUT2: now reaches J3.1 (Pin_1)
- net M3_OUT2: now also D11.1 (K), U6.6 (2Y)
- net M3_OUT1: now reaches J3.2 (Pin_2)
- net M3_OUT1: now also D10.2 (A), U6.3 (1Y)
- net M2_OUT2: now reaches J2.1 (Pin_1)
- net M2_OUT2: now also D8.1 (K), U9.14 (4Y)
- net M2_OUT1: now reaches J2.2 (Pin_2)
- net M2_OUT1: now also D7.2 (A), U9.11 (3Y)
- net M1_OUT2: now reaches J1.1 (Pin_1)
- net M1_OUT2: now also D6.1 (K), U9.6 (2Y)
- net M1_OUT1: now reaches J1.2 (Pin_2)
- net M1_OUT1: now also D5.2 (A), U9.3 (1Y)
- net IN_FC renamed IN_FC1
- net IN_FC1: now also J11.2 (Pin_2); no longer J7.2 (Pin_2)
- net MAN_MCLR: no longer names the net of R7.2, SW1.1
- net MAN_MCLR: now also J6.3 (Pin_3); no longer J6.1 (Pin_1)
- net OUT_FC renamed OUT_FC1
- net OUT_FC1: now also U10.37 (RB4/KBI0/AN9)
- new net: K1.A2, Q1.3 (C)
- new net: C10.2, R15.1, U8.2 (-)
- new net: D9.2 (A2), J14.1 (Pin_1), K1.12
- new net: R18.1, R19.2, U8.3 (+)
- new net: J13.2 (Pin_2), R15.2
- new net: R16.2, R17.1, U8.6 (-)
- new net: R13.2, R14.1, U3.6 (-)
- new net ACTIVACIO_RELE: C13.2, Q1.1 (B), U10.22 (C2IN-/PSP3/RD3)
- new net ANALOGIC_OUT: R19.1, U10.5 (RA3/AN3/Vref+), U8.1
- new net CANH: C6.2, R1.2
- new net CINT_OUT: J10.2 (Pin_2), U10.20 (C1IN-/PSP1/RD1)
- new net GND1: C11.1, C14.1, D11.2 (A), D6.2 (A), D8.2 (A), D9.1 (A1), J14.2 (Pin_2), R9.2
- new net IN_FC2: J7.2 (Pin_2), U3.5 (+)
- new net IN_FC3: J12.2 (Pin_2), U8.5 (+)
- new net M1_BOT: R10.1, SW2.2, U10.34 (RB1/INT1/AN8)
- new net M1_IN1: U10.16 (T1OSI/RC1), U9.2 (1A)
- new net M1_IN2: U10.17 (CCP1/RC2), U9.7 (2A)
- new net M2_BOT: R11.1, SW3.2, U10.33 (RB0/INT0/FLT0/AN10)
- new net M2_IN1: U10.2 (RA0/AN0/CVref), U9.10 (3A)
- new net M2_IN2: U10.3 (RA1/AN1), U9.15 (4A)
- new net M3_BOT: R12.1, SW4.2, U10.6 (RA4/TOCKI)
- new net M3_IN1: U10.4 (RA2/AN2/Vref-), U6.2 (1A)
- new net M3_IN2: U10.38 (RB5/KBI1/PGM), U6.7 (2A)
- new net OUT_FC2: U10.7 (RA5/ANA4/~{SS}/HLVDIN), U3.7
- new net OUT_FC3: U10.19 (C1IN+/PSP0/RD0), U8.7
- new net RELE: U10.21 (C2IN+/PSP2/RD2)
- no-connect marks 18 -> 20
Other:
- added sheet Top (untitled.kicad_sch)
- note added: "08/03/2025"
- note added: "Autors: LaraAlex LavanderaMateo"
- note added: "Botonera"
- note added: "Circuits comparadors pels tres finals de carrera"
- note added: "Config. no inversora de guany 10 per amplificar 450mV que genera el sensor a 45ºC (temp max) a 4,5V."
- note added: "Connexió motors"
- note added: "Cortocircuitar esta resistencia Punto unión masas"
- note added: "DRIVERS"
- note added: "Finals Carrera"
- note added: "Projecte Seients Elèctrics - EdD"
- note added: "RELE"
- note added: "Rev 1.0"
- note added: "Rs connectada a GND s'utilitza en altes freqüències. Volem altes freqs."
- note added: "Sensor de pressió pel cinturó"
- note added: "Sensor temperatura + Condicionament"
- note added: "Transciever CAN mode alta freq"
- note removed: "Circuit comparador per final de carrera"
- note removed: "Final Carrera"
- note removed: "Rs connectada a GND s'utilitza en altes freqüències. Volem altes freqs o més baixes (Rs a 10k-100k)?"
- note removed: "Transciever CAN mode?"
- moved on the sheet: C3, C4, C9, Cadj1, D4, J1, J2, J3, J6, J7, J8, R4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
