File: Projecte_Seients.kicad_sch (KiCad schematic)
At the start: 76 parts, among them J1 Screw_Terminal_01x02, J10 Conn_01x03, J11 Conn_01x02, J12 Conn_01x02, J13 Conn_01x03, J14 Screw_Terminal_01x02, J2 Screw_Terminal_01x02, J3 Screw_Terminal_01x02, J4 Conn_01x05, J5 Conn_01x02, J6 Conn_01x03, J7 Conn_01x02, J8 Conn_01x05, J9 Conn_01x09, K1 Relay_SPDT, Q1 DTC144E, SW1 SW_Push, SW2 SW_Push, SW3 SW_Push, SW4 SW_Push, U1 TJA1051T, U10 PIC18F4580-IP, U3 LM393, U5 24LC512, U6 L293D, U7 LD1086V-DG, U8 LM393, U9 L293D, Y1 Crystal

Commit message: Add files via upload
Parts:
- removed J8: Conn_01x05, Connector_PinHeader_2.54mm:PinHeader_1x05_P2.54mm_Vertical, symbol Connector_Generic:Conn_01x05
- removed J9: Conn_01x09, symbol Connector_Generic:Conn_01x09
- added J8, J9: DE9_Plug, symbol Connector:DE9_Plug
Connections:
- net +5V: now also J8.9, J9.1
- net CANL: now also J8.2, J8.7
- net GND: now also J8.3, J9.5
- net RX: now also J9.2
- net TX: now also J9.3
- no-connect marks 21 -> 26
Other:
- removed sheet Top
- note added: "Bateria"
- note added: "MICROCONTROLADOR"
- note removed: "Està bé?"
- note removed: "Microcontrolador"
- moved on the sheet: C1, C10, C11, C12, C13, C14, C2, C3, C4, C5, C6, C7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

Commit message: Add files via upload
Parts:
- added U2: LT1638CS8_PBF, AlexLibrary:SOIC127P600X175-8N, symbol LT1638CS8_PBF:LT1638CS8_PBF
Connections:
- net +5V: now also U2.8 (V+)
- net ANALOGIC_OUT: now also U2.1 (OUT_A); no longer U8.1
- net GND: now also U2.4 (V-); no longer R18.2
- net at C10.2, R15.1: now also U2.3 (+IN_A); no longer U8.2 (-)
- net at R18.1, R19.2: no longer U8.3 (+)
- new net: R18.2, U2.2 (-IN_A)
- no-connect marks 26 -> 32
Other:
- moved on the sheet: C10, J13, R15, R18, R19, U8A

Commit message: Add files via upload
Parts:
- removed D10, D11: 1N5819, Diode_THT:D_DO-41_SOD81_P10.16mm_Horizontal, symbol Diode:1N5819
- removed D4: LED, LED_SMD:LED_0805_2012Metric, symbol Device:LED
- removed J10, J13: Conn_01x03, symbol Connector_Generic:Conn_01x03
- removed J3: Screw_Terminal_01x02, symbol Connector:Screw_Terminal_01x02
- removed J5: Conn_01x02, Connector_PinHeader_2.54mm:PinHeader_1x02_P2.54mm_Vertical, symbol Connector_Generic:Conn_01x02
- removed U2: LT1638CS8_PBF, AlexLibrary:SOIC127P600X175-8N, symbol LT1638CS8_PBF:LT1638CS8_PBF
- removed U3, U8: LM393, symbol Comparator:LM393
- added C15, C16, C17, C18: 100n, Capacitor_SMD:C_0805_2012Metric, symbol Device:C
- added D10: 1N4007, Diode_THT:D_DO-41_SOD81_P10.16mm_Horizontal, symbol Diode:1N4007
- added D12, D4: 1N5819, Diode_THT:D_DO-41_SOD81_P10.16mm_Horizontal, symbol Diode:1N5819
- added J15, J5: Screw_Terminal_01x02, symbol Connector:Screw_Terminal_01x02
- added R20, R21, R22: 10k, Resistor_SMD:R_0805_2012Metric, symbol Device:R
- added SW5: SW_Push, symbol Switch:SW_Push
- added U2: LM35-D, Package_SO:SOIC-8_3.9x4.9mm_P1.27mm, symbol Sensor_Temperature:LM35-D
- added U3: LT6234, symbol Amplifier_Operational:LT6234
- added U4: LT1721, symbol MateoProjecte:LT1721
- R6: value 150 -> 10k
Connections:
- net +5V: now also R10.2, R11.2, R12.2, R6.2, C15.2, C16.2, C17.2, C18.2, R20.2, R21.2, R22.2, U2.8 (+V_{S}), U3.8 (V+), U4.11, U4.14
- net ANALOGIC_OUT: now also U3.1
- net CINT_OUT: now also R6.1, SW5.2
- net GND: now also J8.4, R18.2, C15.1, C16.1, C17.1, C18.1, J15.1 (Pin_1), SW5.1, U2.4 (GND), U3.4 (V-), U4.3, U4.6; no longer J8.3, R10.2, R11.2, R12.2, R6.2
- net M2_BOT: now also R20.1; no longer R11.1
- net M3_BOT: now also R11.1; no longer R12.1
- net OUT_FC1: now also U4.13
- net OUT_FC2: now also U4.5
- net OUT_FC3: now also U4.4
- net VBAT: now also D10.1 (K), D4.1 (K), J15.2 (Pin_2)
- net at C10.2, R15.1: now also U3.3 (+)
- net at R4.2, R5.1: now also U4.15
- net at R15.2: now also U2.1 (V_{OUT})
- net at R18.1, R19.2: now also U3.2 (-)
- net at R16.2, R17.1: now also U4.2
- net at R13.2, R14.1: now also U4.7
- net CANH: no longer names the net of C6.2, R1.2
- net CANH: now also J8.7
- net CANL: no longer names the net of C7.2, J8.2, R2.1
- net CANL: no longer J8.7
- net GND1 renamed GNDPWR
- net GNDPWR: now also D10.2 (A), D12.2 (A)
- net IN_FC1: no longer names the net of J11.2 (Pin_2)
- net IN_FC1: now also R22.1, U4.16
- net IN_FC2: no longer names the net of J7.2 (Pin_2)
- net IN_FC2: now also R21.1, U4.8
- net IN_FC3: no longer names the net of J12.2 (Pin_2)
- net IN_FC3: now also R12.1, U4.1
- net M1_OUT1: no longer names the net of D5.2 (A), J1.2 (Pin_2)
- net M1_OUT1: now also U9.6 (2Y); no longer U9.3 (1Y)
- net M1_OUT2: no longer names the net of D6.1 (K), J1.1 (Pin_1)
- net M1_OUT2: now also U9.3 (1Y); no longer U9.6 (2Y)
- net M2_OUT1: no longer names the net of D7.2 (A), J2.2 (Pin_2)
- net M2_OUT1: now also D8.1 (K), U9.14 (4Y); no longer U9.11 (3Y)
- removed net M2_OUT2: D8.1 (K), J2.1 (Pin_1), U9.14 (4Y)
- net M3_OUT1: no longer names the net of U6.3 (1Y)
- net M3_OUT1: now also D12.1 (K), J5.1 (Pin_1)
- net M3_OUT2: no longer names the net of U6.6 (2Y)
- net M3_OUT2: now also D4.2 (A), J5.2 (Pin_2)
- net RX: no longer names the net of J9.2, U10.26 (DT/RX/RC7)
- net RXCAN: no longer names the net of U1.4 (RXD), U10.36 (RB3/CANRX)
- net TX: no longer names the net of J9.3, U10.25 (CK/TX/RC6)
- net TXCAN: no longer names the net of U1.1 (TXD), U10.35 (RB2/INT2/CANTX)
- net XTAL1: no longer names the net of C3.1, Y1.1
- net XTAL1: now also U10.13 (OSC1/CLKI/RA7); no longer U10.14 (OSC2/CLKO/RA6)
- net XTAL2: no longer names the net of C4.1, Y1.2
- net XTAL2: now also U10.14 (OSC2/CLKO/RA6); no longer U10.13 (OSC1/CLKI/RA7)
- new net: J2.1 (Pin_1), U9.11 (3Y)
- no-connect marks 32 -> 26
Other:
- note added: "Connectem resistència 120 per evitar reflexions del senyal en la línea. I capacitats de 47nF"
- note removed: "CAN"
- note removed: "Connectem resistència 120 per evitar reflexions del senyal en la línea. I capacitats de desacoplament de 47nF"
- note removed: "Connexió motors"
- note removed: "Finals Carrera"
- note removed: "Usart"
- moved on the sheet: C1, C10, C11, C12, C13, C14, C2, C3, C4, C5, C6, C7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
