File: Projecte_Seients.kicad_sch (KiCad schematic)
At the start: 83 parts, among them J1 Screw_Terminal_01x02, J11 Conn_01x02, J12 Conn_01x02, J14 Screw_Terminal_01x02, J15 Screw_Terminal_01x02, J2 Screw_Terminal_01x02, J4 Conn_01x05, J5 Screw_Terminal_01x02, J6 Conn_01x03, J7 Conn_01x02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

Commit message: Add files via upload
Parts:
- added C19: 100n, Capacitor_SMD:C_0805_2012Metric, symbol Device:C
- U10: footprint Package_DIP:DIP-40_W15.24mm -> Mis_huellas:DIP-40_W15.24mm_SMD
- U4: footprint Package_SO:SOIC-8_3.9x4.9mm_P1.27mm -> Package_SO:SOIC-16_4.55x10.3mm_P1.27mm
- U7: footprint Package_TO_SOT_THT:TO-220-3_Vertical -> Mis_huellas:HuellaDis
Connections:
- net +5V: now also J4.2 (Pin_2), C19.2; no longer J4.4 (Pin_4)
- net GND: now also C19.1
- net M1_BOT: now also U10.7 (RA5/ANA4/~{SS}/HLVDIN); no longer U10.34 (RB1/INT1/AN8)
- net M1_IN1: now also U10.37 (RB4/KBI0/AN9); no longer U10.16 (T1OSI/RC1)
- net M1_IN2: now also U10.33 (RB0/INT0/FLT0/AN10); no longer U10.17 (CCP1/RC2)
- net M2_BOT: now also U10.8 (AN5/~{RD}/RE0); no longer U10.33 (RB0/INT0/FLT0/AN10)
- net M2_IN1: now also U10.34 (RB1/INT1/AN8); no longer U10.2 (RA0/AN0/CVref)
- net M2_IN2: now also U10.38 (RB5/KBI1/PGM); no longer U10.3 (RA1/AN1)
- net M3_BOT: now also U10.9 (C1OUT/AN6/~{WR}/RE1); no longer U10.6 (RA4/TOCKI)
- net M3_IN1: now also U10.29 (P1C/PSP6/RD6); no longer U10.4 (RA2/AN2/Vref-)
- net M3_IN2: now also U10.28 (P1B/PSP5/RD5); no longer U10.38 (RB5/KBI1/PGM)
- net OUT_FC1: now also U10.16 (T1OSI/RC1); no longer U10.37 (RB4/KBI0/AN9)
- net OUT_FC2: now also U10.17 (CCP1/RC2); no longer U10.7 (RA5/ANA4/~{SS}/HLVDIN)
- net PGC: now also J4.5 (Pin_5); no longer J4.1 (Pin_1)
- net PGD: now also J4.4 (Pin_4); no longer J4.2 (Pin_2)
- net PROG_MCLR: now also J4.1 (Pin_1), J6.2 (Pin_2); no longer J4.5 (Pin_5), J6.1 (Pin_1)
- net VBAT: now also K1.5, K1.9; no longer K1.11, K1.A1
- net at U10.1 (~{MCLR}/VPP/RE3): now also J6.1 (Pin_1); no longer J6.2 (Pin_2)
- net at Q1.3 (C): now also K1.9; no longer K1.A2
- net at D9.2 (A2), J14.1 (Pin_1): now also K1.6; no longer K1.12
- net at C6.2, R1.2: now also J8.3; no longer J8.7
- no-connect marks 26 -> 25
Other:
- moved on the sheet: D12, D8, J4

Commit message: Add files via upload
Parts:
- removed U1: TJA1051T, Package_SO:SOIC-8_3.9x4.9mm_P1.27mm, symbol Interface_CAN_LIN:TJA1051T
- added D11, D13, D14, D15, D16, D17: 1N5819, Diode_THT:D_DO-41_SOD81_P10.16mm_Horizontal, symbol Diode:1N5819
- added SW6, SW7, SW8: SW_Push, Mis_huellas:SW_2-1437565-7, symbol Switch:SW_Push
- added TJA1051T1: U1, Package_SO:SOIC-8_3.9x4.9mm_P1.27mm, symbol MateoProjecte:TJA1051T_2
- R9: footprint Resistor_SMD:R_0805_2012Metric -> Resistor_THT:R_Axial_DIN0204_L3.6mm_D1.6mm_P5.08mm_Horizontal
Connections:
- net +5V: now also J4.1 (Pin_1), SW2.1, SW3.1, SW4.1, SW6.1, SW7.1, SW8.1, TJA1051T1.3 (VCC); no longer J4.2 (Pin_2), R10.2, R11.2, R20.2
- net GND: now also R10.2, R11.2, R20.2, TJA1051T1.2 (GND), TJA1051T1.8 (S); no longer SW2.1, SW3.1, SW4.1
- net GNDPWR: now also D13.2 (A), D15.2 (A), D17.2 (A)
- net M1_BOT: now also SW4.2, SW6.2; no longer SW2.2
- net M2_BOT: now also R11.1, SW2.2; no longer R20.1
- net M3_BOT: now also R20.1, SW7.2, SW8.2; no longer R11.1, SW4.2
- net PROG_MCLR: now also J4.2 (Pin_2); no longer J4.1 (Pin_1)
- net VBAT: now also D11.1 (K), D14.1 (K), D16.1 (K)
- net at D12.1 (K), J5.1 (Pin_1), U6.3 (1Y): now also D11.2 (A)
- net at U10.35 (RB2/INT2/CANTX): now also TJA1051T1.1 (TXD)
- net at U10.36 (RB3/CANRX): now also TJA1051T1.4 (RXD)
- net at R2.2: now also TJA1051T1.6 (CAN-)
- net at R1.1: now also TJA1051T1.7 (CAN+)
- net at D4.2 (A), J5.2 (Pin_2), U6.6 (2Y): now also D13.1 (K)
- net at D6.1 (K), J1.1 (Pin_1), U9.3 (1Y): now also D16.2 (A)
- net at D5.2 (A), J1.2 (Pin_2), U9.6 (2Y): now also D17.1 (K)
- net at D7.2 (A), J2.1 (Pin_1), U9.11 (3Y): now also D15.1 (K)
- net at D8.1 (K), J2.2 (Pin_2), U9.14 (4Y): now also D14.2 (A)
Other:
- moved on the sheet: D8, R6, SW5
