File: Projecte_Seients.kicad_pcb (KiCad board)
At the start: 2 copper layers, 83 parts, among them J1 Screw_Terminal_01x02, J11 Conn_01x02, J12 Conn_01x02, J14 Screw_Terminal_01x02, J15 Screw_Terminal_01x02, J2 Screw_Terminal_01x02, J4 Conn_01x05, J5 Screw_Terminal_01x02, J6 Conn_01x03, J7 Conn_01x02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

Commit message: Add files via upload
Parts:
- moved J8 187.9 mm to (202.1, 23.7)
- moved C7 152.5 mm to (189.4, 46.5)
- moved C6 150.3 mm to (220.6, 38.0)
- moved R1 150.3 mm to (220.5, 44.5)
- moved R18 147.2 mm to (117.9, 38.0)
- moved R2 145.1 mm to (196.0, 39.0)
- moved U1 144.3 mm to (202.5, 47.9), turned to 180 degrees
- moved J9 141.1 mm to (129.9, 152.5)
- moved C15 140.0 mm to (176.6, 41.5)
- moved C10 132.7 mm to (120.5, 63.4)
- moved R15 132.7 mm to (113.0, 42.9)
- moved R19 132.7 mm to (120.5, 43.4)
- moved U2 132.7 mm to (108.0, 53.5)
- moved U3 132.7 mm to (128.5, 53.4)
- moved J6 80.0 mm to (162.0, 56.9)
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Connections:
- J4 pad 1: PGC -> PROG_MCLR
- J4 pad 2: PGD -> +5V
- J4 pad 4: +5V -> PGD
- J4 pad 5: PROG_MCLR -> PGC
- J6 pad 1: PROG_MCLR -> Net-(J6-Pin_1)
- J6 pad 2: Net-(J6-Pin_2) -> PROG_MCLR
- U10 pad 1: Net-(J6-Pin_2) -> Net-(J6-Pin_1)
- U10 pad 16: M1_IN1 -> OUT_FC1
- U10 pad 17: M1_IN2 -> OUT_FC2
- U10 pad 2: M2_IN1 -> unconnected-(U10-RA0/AN0/CVref-Pad2)
- U10 pad 28: unconnected-(U10-P1B/PSP5/RD5-Pad28) -> M3_IN2
- U10 pad 29: unconnected-(U10-P1C/PSP6/RD6-Pad29) -> M3_IN1
- U10 pad 3: M2_IN2 -> unconnected-(U10-RA1/AN1-Pad3)
- U10 pad 33: M2_BOT -> M1_IN2
- U10 pad 34: M1_BOT -> M2_IN1
- U10 pad 37: OUT_FC1 -> M1_IN1
- U10 pad 38: M3_IN2 -> M2_IN2
- U10 pad 4: M3_IN1 -> unconnected-(U10-RA2/AN2/Vref--Pad4)
- U10 pad 6: M3_BOT -> unconnected-(U10-RA4/TOCKI-Pad6)
- U10 pad 7: OUT_FC2 -> M1_BOT
- U10 pad 8: unconnected-(U10-AN5/~{RD}/RE0-Pad8) -> M2_BOT
- U10 pad 9: unconnected-(U10-C1OUT/AN6/~{WR}/RE1-Pad9) -> M3_BOT
Routing:
- net +5V: track 0.00 -> 490.6 mm
- net VBAT: track 0.00 -> 144.7 mm
- net M2_IN2: track 0.00 -> 120.3 mm
- net M1_BOT: track 0.00 -> 120.0 mm
- net M2_BOT: track 0.00 -> 115.3 mm
- net OUT_FC3: track 0.00 -> 115.2 mm
- net M1_IN1: track 0.00 -> 114.5 mm
- net OUT_FC2: track 0.00 -> 113.4 mm
- net M3_BOT: track 0.00 -> 110.5 mm
- net OUT_FC1: track 0.00 -> 107.4 mm
- net M2_IN1: track 0.00 -> 97.6 mm
- net M1_IN2: track 0.00 -> 90.1 mm
- net M3_IN1: track 0.00 -> 84.9 mm
- net M3_IN2: track 0.00 -> 80.7 mm
- net ACTIVACIO_RELE: track 0.00 -> 76.6 mm
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
Commit message: Add files via upload
Parts:
- removed R9: 0, Resistor_SMD:R_0805_2012Metric
- added C19: 100n, Capacitor_SMD:C_0805_2012Metric, F.Cu at (200.6, 157.0)
- C12, C9: moved to B.Cu
- moved D10 137.3 mm to (205.8, 54.0)
- moved R1 97.1 mm to (135.0, 90.5)
- moved C11 96.5 mm to (208.1, 47.0)
- moved D2 95.2 mm to (129.6, 28.0)
- moved C6 94.5 mm to (142.0, 90.5), turned to 180 degrees
- moved U1 87.1 mm to (127.5, 92.1), turned to 0 degrees
- moved R3 86.3 mm to (129.6, 102.5)
- moved J8 85.8 mm to (156.0, 96.0), turned to 90 degrees
- moved C16 84.2 mm to (166.1, 55.5)
- moved D4 82.5 mm to (173.4, 83.0)
- moved R2 81.8 mm to (135.0, 93.5), turned to 180 degrees
- moved D3 79.6 mm to (134.6, 102.5)
- moved Q1 79.2 mm to (159.4, 143.0)
- moved C1 76.4 mm to (109.2, 28.0)
- moved C13 76.0 mm to (160.5, 135.5)
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Connections:
- J8 pad 3: unconnected-(J8-Pad3) -> Net-(C6-Pad2)
- J8 pad 7: Net-(C6-Pad2) -> unconnected-(J8-Pad7)
Routing:
- net +5V: track 490.6 -> 65.7 mm, vias 0 -> 6
- net PWM: track 0.00 -> 374.1 mm
- net VBAT: track 144.7 -> 0.00 mm
- net GND: track 15.3 -> 102.0 mm, vias 40 -> 96
- net M1_BOT: track 120.0 -> 47.7 mm
- net M2_BOT: track 115.3 -> 43.7 mm
- net M3_BOT: track 110.5 -> 40.7 mm
- net Net-(U1-RXD): track 52.6 -> 0.00 mm
- net Net-(U1-TXD): track 51.5 -> 0.00 mm
- net OUT_FC1: track 107.4 -> 60.8 mm
- net Net-(D8-K): track 76.4 -> 35.4 mm
- net Net-(U10-DT/RX/RC7): track 60.1 -> 20.0 mm
- net CINT_OUT: track 62.4 -> 25.7 mm
- net PGC: track 43.5 -> 9.73 mm
- net PGD: track 43.5 -> 9.73 mm
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- added copper zone on F.Cu, net +5V
- added copper zone on B.Cu, net GNDPWR
- added copper zone on F.Cu, net VBAT
Other:
- board outline added: 215.5 x 152 mm

Commit message: Add files via upload
Parts:
- removed U1: TJA1051T, Package_SO:SOIC-8_3.9x4.9mm_P1.27mm
- added D11: 1N5819, Diode_THT:D_DO-41_SOD81_P10.16mm_Horizontal, F.Cu at (222.9, 91.5)
- added D13: 1N5819, Diode_THT:D_DO-41_SOD81_P10.16mm_Horizontal, F.Cu at (215.5, 90.0)
- added D14: 1N5819, Diode_THT:D_DO-41_SOD81_P10.16mm_Horizontal, F.Cu at (217.8, 26.5)
- added D15: 1N5819, Diode_THT:D_DO-41_SOD81_P10.16mm_Horizontal, F.Cu at (232.0, 48.0)
- added D16: 1N5819, Diode_THT:D_DO-41_SOD81_P10.16mm_Horizontal, F.Cu at (241.1, 21.0)
- added D17: 1N5819, Diode_THT:D_DO-41_SOD81_P10.16mm_Horizontal, F.Cu at (217.5, 43.5)
- added R9: 0, Resistor_THT:R_Axial_DIN0204_L3.6mm_D1.6mm_P5.08mm_Horizontal, F.Cu at (205.3, 109.1)
- added REF**: MountingHole_3.2mm_M3, MountingHole:MountingHole_3.2mm_M3, F.Cu at (38.0, 20.0)
- added REF**: MountingHole_3.2mm_M3, MountingHole:MountingHole_3.2mm_M3, F.Cu at (242.5, 161.0)
- added SW6: SW_Push, Mis_huellas:SW_2-1437565-7, F.Cu at (55.5, 75.8)
- added SW7: SW_Push, Mis_huellas:SW_2-1437565-7, F.Cu at (55.5, 95.5)
- added SW8: SW_Push, Mis_huellas:SW_2-1437565-7, F.Cu at (79.0, 93.8)
- added TJA1051T1: U1, Package_SO:SOIC-8_3.9x4.9mm_P1.27mm, F.Cu at (129.5, 92.0)
- moved D5 67.2 mm to (243.0, 44.9), turned to -90 degrees
- moved D12 49.3 mm to (233.0, 97.5)
- moved D4 38.5 mm to (211.9, 82.5)
- moved C19 36.5 mm to (164.1, 158.5)
- moved C16 26.1 mm to (192.1, 53.0)
- moved SW3 23.6 mm to (55.5, 85.8)
- moved SW4 19.8 mm to (79.0, 74.2)
- moved C18 16.2 mm to (197.6, 58.5)
- moved R20 11.0 mm to (68.5, 94.9), turned to -90 degrees
- moved SW2 9.75 mm to (79.0, 84.0)
- moved R11 9.15 mm to (68.5, 84.9), turned to -90 degrees
- moved J1 6.52 mm to (233.5, 53.5)
- moved C11 5.95 mm to (213.4, 49.5), turned to 180 degrees
- moved D8 5.10 mm to (207.4, 31.5)
- moved D10 4.35 mm to (209.9, 55.5)
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Connections:
- J4 pad 1: PROG_MCLR -> +5V
- J4 pad 2: +5V -> PROG_MCLR
- R10 pad 2: +5V -> GND
- R11 pad 1: M3_BOT -> M2_BOT
- R11 pad 2: +5V -> GND
- R20 pad 1: M2_BOT -> M3_BOT
- R20 pad 2: +5V -> GND
- SW2 pad 1: GND -> +5V
- SW2 pad 2: M1_BOT -> M2_BOT
- SW3 pad 1: GND -> +5V
- SW4 pad 1: GND -> +5V
- SW4 pad 2: M3_BOT -> M1_BOT
Routing:
- net VBAT: track 0.00 -> 86.4 mm, vias 0 -> 6
- net +5V: track 65.7 -> 130.3 mm, vias 6 -> 10
- net Net-(D11-A): track 43.1 -> 65.5 mm
- net PWM: track 374.1 -> 388.9 mm
- net GND: track 102.0 -> 114.6 mm, vias 96 -> 98
- net Net-(D16-A): track 72.6 -> 85.0 mm
- net M3_BOT: track 40.7 -> 53.2 mm
- net M3_IN2: track 91.7 -> 103.6 mm
- net Net-(D15-K): track 37.5 -> 49.0 mm
- net M2_BOT: track 43.7 -> 54.9 mm
- net M1_BOT: track 47.7 -> 58.9 mm
- net Net-(D17-K): track 54.3 -> 63.3 mm
- net Net-(TJA1051T1-TXD): track 0.00 -> 7.85 mm
- net Net-(TJA1051T1-RXD): track 0.00 -> 7.75 mm
- net GNDPWR: track 6.17 -> 13.6 mm
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